File: electrical/PCB design (KiCAD)/TMotor_Rev0_5_1_Mark_2_NAU_OpenExo_1.kicad_sch (KiCad schematic)
At the start: 11 parts, among them J1 Conn_01x07_Pin, U1 TXU0104PWR, U10 DEV-16771, U2 TXU0304-Q1

Commit message: 26/06 schematics updates
see the changelog on the documentation /electrical/pcb
Parts:
- added TeensyPowerJP1: SolderJumper_2_Open, Jumper:SolderJumper-2_P1.3mm_Open_RoundedPad1.0x1.5mm, symbol Jumper:SolderJumper_2_Open
- renumbered JP6 to CSVoltageShifterOEJP1, JP7 to SPIVoltageShifterOEJP1
Connections:
- net +5V: now also TeensyPowerJP1.1 (A); no longer U10.VIN
- new net: TeensyPowerJP1.2 (B), U10.VIN
Changed lines of the file:
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@@
 	(wire
 		(pts
-			(xy 172.72 66.04) (xy 162.56 66.04)
+			(xy 172.72 66.04) (xy 168.91 66.04)
 		)
 		(stroke
@@
 	(wire
 		(pts
+			(xy 154.94 66.04) (xy 161.29 66.04)
+		)
+		(stroke
+			(width 0.1524)
+			(type solid)
+		)
+	)
+	(wire
+		(pts
 			(xy 105.41 15.24) (xy 107.95 15.24)
 		)
@@
 	(wire
 		(pts
+			(xy 154.94 60.96) (xy 154.94 66.04)
+		)
+		(stroke
+			(width 0.1524)
+			(type solid)
+		)
+	)
+	(wire
+		(pts
 			(xy 86.36 139.7) (xy 78.74 139.7)
 		)
@@
 		(on_board yes)
 		(dnp no)
-		(fields_autoplaced yes)
-		(property "Reference" "JP7"
-			(at 139.7 76.2001 90)
+		(property "Reference" "SPIVoltageShifterOEJP1"
+			(at 138.684 72.644 90)
 			(effects
 				(font
@@
 		)
 		(property "Value" "SolderJumper_3_Open"
-			(at 139.7 73.6601 90)
+			(at 138.938 74.676 90)
 			(effects
 				(font
@@
 			(project "TMotor_Rev0_5_1_Mark_2_NAU_OpenExo"
 				(path "/3e3ff72e-d777-45cf-9299-e91389ff12dd/488ec729-0dfb-4444-ad76-08976c45f4bf"
-					(reference "JP7")
+					(reference "SPIVoltageShifterOEJP1")
 					(unit 1)
 				)
@@
 		(dnp no)
 		(fields_autoplaced yes)
-		(property "Reference" "JP6"
+		(property "Reference" "CSVoltageShifterOEJP1"
 			(at 39.37 21.5899 90)
 			(effects
@@
 			(project ""
 				(path "/3e3ff72e-d777-45cf-9299-e91389ff12dd/488ec729-0dfb-4444-ad76-08976c45f4bf"
-					(reference "JP6")
+					(reference "CSVoltageShifterOEJP1")
 					(unit 1)
 				)
@@
 	)
 	(symbol
+		(lib_id "Jumper:SolderJumper_2_Open")
+		(at 165.1 66.04 0)
+		(unit 1)
+		(exclude_from_sim no)
+		(in_bom no)
+		(on_board yes)
+		(dnp no)
+		(property "Reference" "TeensyPowerJP1"
+			(at 165.1 59.69 0)
+			(effects
+				(font
+					(size 1.27 1.27)
+				)
+			)
+		)
+		(property "Value" "SolderJumper_2_Open"
+			(at 166.37 62.23 0)
+			(effects
+				(font
+					(size 1.27 1.27)
+				)
+			)
+		)
+		(property "Footprint" "Jumper:SolderJumper-2_P1.3mm_Open_RoundedPad1.0x1.5mm"
+			(at 165.1 66.04 0)
+			(effects
+				(font
+					(size 1.27 1.27)
+				)
+				(hide yes)
+			)
+		)
+		(property "Datasheet" "~"
+			(at 165.1 66.04 0)
+			(effects
+				(font
+					(size 1.27 1.27)
+				)
+				(hide yes)
+			)
+		)
+		(property "Description" "Solder Jumper, 2-pole, open"
+			(at 165.1 66.04 0)
+			(effects
+				(font
+					(size 1.27 1.27)
+				)
+				(hide yes)
+			)
+		)
+		(pin "1"
+		)
+		(pin "2"
+		)
+		(instances
+			(project ""
+				(path "/3e3ff72e-d777-45cf-9299-e91389ff12dd/488ec729-0dfb-4444-ad76-08976c45f4bf"
+					(reference "TeensyPowerJP1")
+					(unit 1)
+				)
+			)
+		)
+	)
+	(symbol
 		(lib_id "power:GND")
 		(at 105.41 20.32 0)
@@
 	(symbol
 		(lib_id "power:+5V")
-		(at 162.56 66.04 0)
+		(at 154.94 60.96 0)
 		(unit 1)
 		(exclude_from_sim no)
@@
 		(fields_autoplaced yes)
 		(property "Reference" "#PWR026"
-			(at 162.56 69.85 0)
+			(at 154.94 64.77 0)
 			(effects
 				(font
@@
 		)
 		(property "Value" "+5V"
-			(at 162.56 60.96 0)
+			(at 154.94 55.88 0)
 			(effects
 				(font
@@
 		)
 		(property "Footprint" ""
-			(at 162.56 66.04 0)
+			(at 154.94 60.96 0)
 			(effects
 				(font
@@
 		)
 		(property "Datasheet" ""
-			(at 162.56 66.04 0)
+			(at 154.94 60.96 0)
 			(effects
 				(font
@@
 		)
 		(property "Description" "Power symbol creates a global label with name \"+5V\""
-			(at 162.56 66.04 0)
+			(at 154.94 60.96 0)
 			(effects
 				(font
