File: electrical/PCB design (KiCAD)/TMotor_Rev0_5_1_Mark_2_NAU_OpenExo.kicad_pcb (KiCad board)
At the start: 2 copper layers, 89.4 x 82.6 mm, 118 parts, among them J10 XT30PW-F, J11 XT30PW-F, J2 Conn_01x04_Pin, J3 Conn_01x02_Pin, J4 Conn_01x02_Pin, J5 Conn_01x02_Pin, J6 Conn_01x03_Pin, J7 XT30PW-F, J8 XT30PW-F, J9 XT30PW-F, U1 INA125U, U10 INA232AIDDFR, U2 INA125U, U3 INA125U, U4 INA125U, U5 TXU0104PWR, U6 TXU0304-Q1, U7 DEV-16771, U8 SN65HVD230DR, U9 WPME-FDSM_SIP-3

Commit message: updates
Parts:
- removed J6: Conn_01x03_Pin, Connector_PinHeader_2.54mm:PinHeader_1x03_P2.54mm_Vertical
- added J1: Conn_02x03_Counter_Clockwise, Connector_PinHeader_2.54mm:PinHeader_2x03_P2.54mm_Vertical, F.Cu at (174.9, 77.7)
Routing:
- net GND: track 29.8 -> 33.0 mm
- net /CAN and peripherals./CAN_P: track 113.0 -> 114.6 mm
- net /CAN and peripherals./CAN_N: track 113.6 -> 115.2 mm
- net SHIELD: track 246.8 -> 248.3 mm
Other:
- outline, holes or cut-outs redrawn
