File: electrical/PCB design (KiCAD)/TMotor_Rev0_5_1_Mark_2_NAU_OpenExo_2.kicad_sch (KiCad schematic)
At the start: 30 parts, among them J10 XT30PW-F, J11 XT30PW-F, J12 XT30PW-F, J2 Conn_01x04_Pin, J3 Conn_01x02_Pin, J4 Conn_01x02_Pin, J5 Conn_01x02_Pin, J6 Conn_01x02_Pin, J7 Conn_01x03_Pin, J8 XT30PW-F, J9 XT30PW-F, U5 SN65HVD230DR

Commit message: documentation update for my 10 days leave ; documentation for first time teensy setup on Arduino IDE ;  SW revamp to use HW versioning conditional compiling
Parts:
- added D6: LED, LED_SMD:LED_0805_2012Metric, symbol Device:LED
- added R7: 600kR, Resistor_THT:R_Axial_DIN0207_L6.3mm_D2.5mm_P10.16mm_Horizontal, symbol TMotor_Rev0_5_1_Mark_2_NAU_OpenExo-eagle-import:R-US_0207/10
- added TP1, TP2: TestPoint, TestPoint:TestPoint_Keystone_5000-5004_Miniature, symbol Connector:TestPoint
Connections:
- net +5V: now also R7.2
- net CANRX: now also TP1.1
- net CANTX: now also TP2.1
- net GND: now also D6.1 (K)
- new net: D6.2 (A), R7.1

Commit message: design updates ; documentation update
Parts:
- removed C15, C3: 100nF, Capacitor_THT:C_Disc_D10.5mm_W5.0mm_P5.00mm, symbol TMotor_Rev0_5_1_Mark_2_NAU_OpenExo-eagle-import:C-EU050-024X044
- removed J10, J11, J12, J8, J9: XT30PW-F, XT30PW-F:AMASS_XT30U-F_1x02_P5.0mm_Vertical, symbol XT30PW-F:XT30PW-F
- removed J4: Conn_01x02_Pin, Connector_PinHeader_2.54mm:PinHeader_1x02_P2.54mm_Vertical, symbol Connector:Conn_01x02_Pin
- removed PS1: P78E05-1000, TMotor_Rev0_5_1_Mark_2_NAU_OpenExo:P78E05-1000, symbol P78E05-1000:P78E05-1000
- added C10, C11: 22uF, Capacitor_SMD:C_0805_2012Metric_Pad1.18x1.45mm_HandSolder, symbol Device:C
- added J10, J11, J7, J8, J9: XT30PW-F, XT30 new version:AMASS_XT30U-F_1x02_P5.0mm_Vertical, symbol XT30 conn:XT30PW-F
- added U9: WPME-FDSM_SIP-3, 173010535:WPME-FDSM_17301XX35, symbol 173010535:WPME-FDSM_SIP-3
- C5: renamed from C23; footprint Capacitor_THT:C_Disc_D10.5mm_W5.0mm_P5.00mm -> Capacitor_SMD:C_0805_2012Metric_Pad1.18x1.45mm_HandSolder
- C6: renamed from C5; footprint Capacitor_THT:C_Disc_D10.5mm_W5.0mm_P5.00mm -> Capacitor_SMD:C_0805_2012Metric_Pad1.18x1.45mm_HandSolder
- C7: renamed from C9; footprint Capacitor_THT:C_Disc_D10.5mm_W5.0mm_P5.00mm -> Capacitor_SMD:C_0805_2012Metric_Pad1.18x1.45mm_HandSolder
- C9: renamed from C4; footprint Capacitor_THT:C_Disc_D10.5mm_W5.0mm_P5.00mm -> Capacitor_SMD:C_0805_2012Metric_Pad1.18x1.45mm_HandSolder
- R1: renamed from R12; footprint Resistor_THT:R_Axial_DIN0207_L6.3mm_D2.5mm_P10.16mm_Horizontal -> Resistor_SMD:R_0805_2012Metric_Pad1.20x1.40mm_HandSolder
- R2: renamed from R1; footprint Resistor_THT:R_Axial_DIN0207_L6.3mm_D2.5mm_P10.16mm_Horizontal -> Resistor_SMD:R_0805_2012Metric_Pad1.20x1.40mm_HandSolder
- R3: renamed from R2; value 10R -> 10; footprint Resistor_THT:R_Axial_DIN0207_L6.3mm_D2.5mm_P10.16mm_Horizontal -> Resistor_SMD:R_0805_2012Metric_Pad1.20x1.40mm_HandSolder
- R4: renamed from R11; footprint Resistor_THT:R_Axial_DIN0207_L6.3mm_D2.5mm_P10.16mm_Horizontal -> Resistor_SMD:R_0805_2012Metric_Pad1.20x1.40mm_HandSolder
- R5: renamed from R7; footprint Resistor_THT:R_Axial_DIN0207_L6.3mm_D2.5mm_P10.16mm_Horizontal -> Resistor_SMD:R_0805_2012Metric_Pad1.20x1.40mm_HandSolder
- renumbered C1 to C8, D2 to D1, D6 to D2, INA219 to INA1, J6 to J3, J5 to J4, J3 to J5, J7 to J6, SHUNT0 to SHUNT1, TP2 to TP1, TP1 to TP2, U$6 to U$1, U5 to U8
Connections:
- net GND: now also C10.2, C11.2, J10.1 (-), J11.1 (-), J7.1 (-), J8.1 (-), J9.1 (-), U9.2
- net L7_VIN: now also U9.1
- net VBATT: now also J10.2 (+), J11.2 (+), J7.2 (+), J8.2 (+), J9.2 (+)
- net at U$1.1 (P$1): now also C10.1, C11.1, U9.3
Other:
- moved on the sheet: D2, R5

Commit message: updated ble and uart
Parts:
- removed R5: 600kR, Resistor_SMD:R_0805_2012Metric_Pad1.20x1.40mm_HandSolder, symbol TMotor_Rev0_5_1_Mark_2_NAU_OpenExo-eagle-import:R-US_0207/10
- added C12: 100nF, Capacitor_SMD:C_0805_2012Metric_Pad1.18x1.45mm_HandSolder, symbol TMotor_Rev0_5_1_Mark_2_NAU_OpenExo-eagle-import:C-EU050-024X044
- added R5: 1k, Resistor_SMD:R_0805_2012Metric_Pad1.20x1.40mm_HandSolder, symbol Device:R
Connections:
- net +3V3: now also C12.1
- net +5V: now also R5.1
- net GND: now also C12.2
- net at D2.2 (A): now also R5.2
Changed lines of the file:
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@@
 	)
 	(junction
+		(at 303.53 180.34)
+		(diameter 0)
+		(color 0 0 0 0)
+	)
+	(junction
 		(at 129.54 261.62)
 		(diameter 0)
@@
 	)
 	(junction
-		(at 38.1 167.64)
+		(at 81.28 236.22)
 		(diameter 0)
 		(color 0 0 0 0)
 	)
 	(junction
-		(at 269.24 96.52)
+		(at 38.1 167.64)
 		(diameter 0)
 		(color 0 0 0 0)
 	)
 	(junction
-		(at 303.53 180.34)
+		(at 269.24 96.52)
 		(diameter 0)
 		(color 0 0 0 0)
@@
 	(wire
 		(pts
-			(xy 303.53 191.77) (xy 303.53 190.5)
+			(xy 303.53 189.23) (xy 303.53 191.77)
 		)
 		(stroke
@@
 	(wire
 		(pts
+			(xy 81.28 236.22) (xy 81.28 251.46)
+		)
+		(stroke
+			(width 0.1524)
+			(type solid)
+		)
+	)
+	(wire
+		(pts
 			(xy 346.71 74.93) (xy 346.71 96.52)
 		)
@@
 	(wire
 		(pts
-			(xy 81.28 251.46) (xy 83.82 251.46)
-		)
-		(stroke
-			(width 0.1524)
-			(type solid)
-		)
-	)
-	(wire
-		(pts
 			(xy 43.18 147.32) (xy 35.56 147.32)
 		)
@@
 	(wire
 		(pts
+			(xy 81.28 236.22) (xy 90.17 236.22)
+		)
+		(stroke
+			(width 0)
+			(type default)
+		)
+	)
+	(wire
+		(pts
 			(xy 200.66 147.32) (xy 200.66 132.08)
 		)
@@
 	(wire
 		(pts
+			(xy 81.28 234.95) (xy 81.28 236.22)
+		)
+		(stroke
+			(width 0.1524)
+			(type solid)
+		)
+	)
+	(wire
+		(pts
 			(xy 86.36 271.78) (xy 86.36 279.4)
 		)
@@
 	(wire
 		(pts
+			(xy 303.53 180.34) (xy 303.53 181.61)
+		)
+		(stroke
+			(width 0)
+			(type default)
+		)
+	)
+	(wire
+		(pts
 			(xy 45.72 256.54) (xy 40.64 256.54)
 		)
@@
 	(symbol
 		(lib_id "power:+3V3")
-		(at 83.82 251.46 0)
+		(at 81.28 234.95 0)
 		(unit 1)
 		(exclude_from_sim no)
@@
 		(on_board yes)
 		(dnp no)
-		(fields_autoplaced yes)
 		(property "Reference" "#PWR024"
-			(at 83.82 255.27 0)
+			(at 81.28 238.76 0)
 			(effects
 				(font
@@
 		)
 		(property "Value" "+3V3"
-			(at 83.82 246.38 0)
+			(at 85.09 233.68 0)
 			(effects
 				(font
@@
 		)
 		(property "Footprint" ""
-			(at 83.82 251.46 0)
+			(at 81.28 234.95 0)
 			(effects
 				(font
@@
 		)
 		(property "Datasheet" ""
-			(at 83.82 251.46 0)
+			(at 81.28 234.95 0)
 			(effects
 				(font
@@
 		)
 		(property "Description" "Power symbol creates a global label with name \"+3V3\""
-			(at 83.82 251.46 0)
+			(at 81.28 234.95 0)
 			(effects
 				(font
@@
 	)
 	(symbol
+		(lib_id "Device:R")
+		(at 303.53 185.42 0)
+		(unit 1)
+		(exclude_from_sim no)
+		(in_bom yes)
+		(on_board yes)
+		(dnp no)
+		(fields_autoplaced yes)
+		(property "Reference" "R5"
+			(at 306.07 184.1499 0)
+			(effects
+				(font
+					(size 1.27 1.27)
+				)
+				(justify left)
+			)
+		)
+		(property "Value" "1k"
+			(at 306.07 186.6899 0)
+			(effects
+				(font
+					(size 1.27 1.27)
+				)
+				(justify left)
+			)
+		)
+		(property "Footprint" "Resistor_SMD:R_0805_2012Metric_Pad1.20x1.40mm_HandSolder"
+			(at 301.752 185.42 90)
+			(effects
+				(font
+					(size 1.27 1.27)
+				)
+				(hide yes)
+			)
+		)
+		(property "Datasheet" "~"
+			(at 303.53 185.42 0)
+			(effects
+				(font
+					(size 1.27 1.27)
+				)
+				(hide yes)
+			)
+		)
+		(property "Description" "Resistor"
+			(at 303.53 185.42 0)
+			(effects
+				(font
+					(size 1.27 1.27)
+				)
+				(hide yes)
+			)
+		)
+		(pin "1"
+		)
+		(pin "2"
+		)
+		(instances
+			(project ""
+				(path "/3e3ff72e-d777-45cf-9299-e91389ff12dd/ec3a94af-cbf2-4645-8611-15dc332be977"
+					(reference "R5")
+					(unit 1)
+				)
+			)
+		)
+	)
+	(symbol
 		(lib_id "TMotor_Rev0_5_1_Mark_2_NAU_OpenExo-eagle-import:R-US_0207/10")
 		(at 203.2 261.62 90)
@@
 	(symbol
 		(lib_id "TMotor_Rev0_5_1_Mark_2_NAU_OpenExo-eagle-import:R-US_0207/10")
-		(at 303.53 185.42 90)
-		(unit 1)
-		(exclude_from_sim no)
-		(in_bom yes)
-		(on_board yes)
-		(dnp no)
-		(property "Reference" "R5"
-			(at 302.0314 189.23 0)
-			(effects
-				(font
-					(size 1.778 1.5113)
-				)
-				(justify left bottom)
-			)
-		)
-		(property "Value" "600kR"
-			(at 306.832 189.23 0)
-			(effects
-				(font
-					(size 1.778 1.5113)
-				)
-				(justify left bottom)
-			)
-		)
-		(property "Footprint" "Resistor_SMD:R_0805_2012Metric_Pad1.20x1.40mm_HandSolder"
-			(at 303.53 185.42 0)
-			(effects
-				(font
-					(size 1.27 1.27)
-				)
-				(hide yes)
-			)
-		)
-		(property "Datasheet" ""
-			(at 303.53 185.42 0)
-			(effects
-				(font
-					(size 1.27 1.27)
-				)
-				(hide yes)
-			)
-		)
-		(property "Description" ""
-			(at 303.53 185.42 0)
-			(effects
-				(font
-					(size 1.27 1.27)
-				)
-				(hide yes)
-			)
-		)
-		(pin "1"
-		)
-		(pin "2"
-		)
-		(instances
-			(project "TMotor_Rev0_5_1_Mark_2_NAU_OpenExo"
-				(path "/3e3ff72e-d777-45cf-9299-e91389ff12dd/ec3a94af-cbf2-4645-8611-15dc332be977"
-					(reference "R5")
-					(unit 1)
-				)
-			)
-		)
-	)
-	(symbol
-		(lib_id "TMotor_Rev0_5_1_Mark_2_NAU_OpenExo-eagle-import:R-US_0207/10")
 		(at 101.6 248.92 180)
 		(unit 1)
@@
 					(unit 1)
 				)
+			)
+		)
+	)
+	(symbol
+		(lib_id "TMotor_Rev0_5_1_Mark_2_NAU_OpenExo-eagle-import:C-EU050-024X044")
+		(at 90.17 238.76 0)
+		(mirror y)
+		(unit 1)
+		(exclude_from_sim no)
+		(in_bom yes)
+		(on_board yes)
+		(dnp no)
+		(property "Reference" "C12"
+			(at 88.646 238.379 0)
+			(effects
+				(font
+					(size 1.778 1.5113)
+				)
+				(justify left bottom)
+			)
+		)
+		(property "Value" "100nF"
+			(at 100.584 241.808 0)
+			(effects
+				(font
+					(size 1.778 1.5113)
+				)
+				(justify left bottom)
+			)
+		)
+		(property "Footprint" "Capacitor_SMD:C_0805_2012Metric_Pad1.18x1.45mm_HandSolder"
+			(at 90.17 238.76 0)
+			(effects
+				(font
+					(size 1.27 1.27)
+				)
+				(hide yes)
+			)
+		)
+		(property "Datasheet" ""
+			(at 90.17 238.76 0)
+			(effects
+				(font
+					(size 1.27 1.27)
+				)
+				(hide yes)
+			)
+		)
+		(property "Description" ""
+			(at 90.17 238.76 0)
+			(effects
+				(font
+					(size 1.27 1.27)
+				)
+				(hide yes)
+			)
+		)
+		(pin "1"
+		)
+		(pin "2"
+		)
+		(instances
+			(project "TMotor_Rev0_5_1_Mark_2_NAU_OpenExo"
+				(path "/3e3ff72e-d777-45cf-9299-e91389ff12dd/ec3a94af-cbf2-4645-8611-15dc332be977"
+					(reference "C12")
+					(unit 1)
+				)
+			)
+		)
+	)
+	(symbol
+		(lib_id "power:GND")
+		(at 90.17 243.84 0)
+		(unit 1)
+		(exclude_from_sim no)
+		(in_bom yes)
+		(on_board yes)
+		(dnp no)
+		(fields_autoplaced yes)
+		(property "Reference" "#PWR043"
+			(at 90.17 250.19 0)
+			(effects
+				(font
+					(size 1.27 1.27)
+				)
+				(hide yes)
+			)
+		)
+		(property "Value" "GND"
+			(at 90.17 248.92 0)
+			(effects
+				(font
+					(size 1.27 1.27)
+				)
+			)
+		)
+		(property "Footprint" ""
+			(at 90.17 243.84 0)
+			(effects
+				(font
+					(size 1.27 1.27)
+				)
+				(hide yes)
+			)
+		)
+		(property "Datasheet" ""
+			(at 90.17 243.84 0)
+			(effects
+				(font
+					(size 1.27 1.27)
+				)
+				(hide yes)
+			)
+		)
+		(property "Description" "Power symbol creates a global label with name \"GND\" , ground"
+			(at 90.17 243.84 0)
+			(effects
+				(font
+					(size 1.27 1.27)
+				)
+				(hide yes)
+			)
+		)
+		(pin "1"
+		)
+		(instances
+			(project "TMotor_Rev0_5_1_Mark_2_NAU_OpenExo"
+				(path "/3e3ff72e-d777-45cf-9299-e91389ff12dd/ec3a94af-cbf2-4645-8611-15dc332be977"
+					(reference "#PWR043")
+					(unit 1)
+				)

Commit message: updates
Parts:
- removed C6: 100nF, Capacitor_SMD:C_0805_2012Metric_Pad1.18x1.45mm_HandSolder, symbol TMotor_Rev0_5_1_Mark_2_NAU_OpenExo-eagle-import:C-EU050-024X044
- removed INA1: ~, TMotor_Rev0_5_1_Mark_2_NAU_OpenExo:D8_TEX, symbol TMotor_Rev0_5_1_Mark_2_NAU_OpenExo-eagle-import:INA219AIDR
- added C17: 0.1uF, Capacitor_SMD:C_0805_2012Metric_Pad1.18x1.45mm_HandSolder, symbol TMotor_Rev0_5_1_Mark_2_NAU_OpenExo-eagle-import:C-EU050-024X044
- added R27, R28: 3.3k, Resistor_SMD:R_0805_2012Metric_Pad1.20x1.40mm_HandSolder, symbol Device:R
- added U10: INA232AIDDFR, SOT_32AIDDFR_TEX, symbol INA232AIDDFR:INA232AIDDFR
- C7: value 100nF -> 0.1uF
- R2: value 10R -> 10
Connections:
- net +3V3: now also C17.2, R27.1, R28.1, U10.4 (VS)
- net GND: now also C17.1, U10.3 (GND), U10.7 (A0)
- net SCL: now also R28.2, U10.5 (SCL)
- net SDA: now also R27.2, U10.6 (SDA)
- net at C7.2, R2.1: now also U10.2 (IN-)
- net at C7.1, R3.1: now also U10.1 (IN+)
- no-connect marks 1 -> 2
Other:
- note removed: "Here is to measure the battery voltage. INA219 is a sensor that will use the info from pins VIN+ and VIN- to estimate the voltage of the power supply. INA219 requires an external SHUNT circuit as shown here."
- note removed: "VS: Power supply for the INA 219 sensor (INA 219 takes 3 to 5.5 V) GND: Ground for the INA 219 sensor"

Commit message: updates
Parts:
- removed J6: Conn_01x03_Pin, Connector_PinHeader_2.54mm:PinHeader_1x03_P2.54mm_Vertical, symbol Connector:Conn_01x03_Pin
- added J1: Conn_02x03_Counter_Clockwise, Connector_PinHeader_2.54mm:PinHeader_2x03_P2.54mm_Vertical, symbol Connector_Generic:Conn_02x03_Counter_Clockwise
Connections:
- net CAN_N: now also J1.3 (Pin_3), J1.4 (Pin_4)
- net CAN_P: now also J1.5 (Pin_5), J1.6 (Pin_6)
- net GND: now also J1.1 (Pin_1), J1.2 (Pin_2)
Changed lines of the file:
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@@
 	(wire
 		(pts
-			(xy 100.33 207.01) (xy 92.71 207.01)
-		)
-		(stroke
-			(width 0.1524)
-			(type solid)
-		)
-	)
-	(wire
-		(pts
 			(xy 307.34 74.93) (xy 307.34 83.82)
 		)
@@
 	(wire
 		(pts
-			(xy 100.33 212.09) (xy 88.9 212.09)
-		)
-		(stroke
-			(width 0)
-			(type default)
-		)
-	)
-	(wire
-		(pts
 			(xy 190.5 266.7) (xy 203.2 266.7)
 		)
@@
 	(wire
 		(pts
+			(xy 91.44 209.55) (xy 92.71 209.55)
+		)
+		(stroke
+			(width 0)
+			(type default)
+		)
+	)
+	(wire
+		(pts
 			(xy 128.27 154.94) (xy 128.27 157.48)
 		)
@@
 	(wire
 		(pts
+			(xy 88.9 207.01) (xy 100.33 207.01)
+		)
+		(stroke
+			(width 0.1524)
+			(type solid)
+		)
+	)
+	(wire
+		(pts
 			(xy 303.53 199.39) (xy 303.53 203.2)
 		)
@@
 	(wire
 		(pts
+			(xy 119.38 207.01) (xy 113.03 207.01)
+		)
+		(stroke
+			(width 0)
+			(type default)
+		)
+	)
+	(wire
+		(pts
 			(xy 132.08 264.16) (xy 132.08 261.62)
 		)
@@
 	(wire
 		(pts
+			(xy 113.03 209.55) (xy 119.38 209.55)
+		)
+		(stroke
+			(width 0)
+			(type default)
+		)
+	)
+	(wire
+		(pts
 			(xy 269.24 96.52) (xy 309.88 96.52)
 		)
@@
 	(wire
 		(pts
+			(xy 92.71 212.09) (xy 100.33 212.09)
+		)
+		(stroke
+			(width 0)
+			(type default)
+		)
+	)
+	(wire
+		(pts
 			(xy 35.56 190.5) (xy 43.18 190.5)
 		)
@@
 	(wire
 		(pts
-			(xy 88.9 212.09) (xy 88.9 213.36)
+			(xy 88.9 207.01) (xy 88.9 213.36)
 		)
 		(stroke
@@
 	(wire
 		(pts
+			(xy 119.38 212.09) (xy 113.03 212.09)
+		)
+		(stroke
+			(width 0)
+			(type default)
+		)
+	)
+	(wire
+		(pts
 			(xy 96.52 248.92) (xy 96.52 256.54)
 		)
@@
 	(wire
 		(pts
+			(xy 91.44 209.55) (xy 91.44 218.44)
+		)
+		(stroke
+			(width 0)
+			(type default)
+		)
+	)
+	(wire
+		(pts
 			(xy 167.64 182.88) (xy 185.42 182.88)
 		)
@@
 	)
 	(label "CAN_P"
-		(at 92.71 207.01 0)
+		(at 119.38 207.01 180)
 		(effects
 			(font
 				(size 1.27 1.27)
 			)
-			(justify left bottom)
+			(justify right bottom)
 		)
 	)
 	(label "CAN_N"
-		(at 92.71 209.55 0)
+		(at 119.38 212.09 180)
+		(effects
+			(font
+				(size 1.27 1.27)
+			)
+			(justify right bottom)
+		)
+	)
+	(label "CAN_N"
+		(at 92.71 212.09 0)
 		(effects
 			(font
@@
 		)
 	)
+	(label "CAN_P"
+		(at 119.38 209.55 180)
+		(effects
+			(font
+				(size 1.27 1.27)
+			)
+			(justify right bottom)
+		)
+	)
 	(global_label "RESET"
 		(shape bidirectional)
@@
 	)
 	(symbol
+		(lib_id "Connector_Generic:Conn_02x03_Counter_Clockwise")
+		(at 105.41 209.55 0)
+		(unit 1)
+		(exclude_from_sim no)
+		(in_bom yes)
+		(on_board yes)
+		(dnp no)
+		(fields_autoplaced yes)
+		(property "Reference" "J1"
+			(at 106.68 200.66 0)
+			(effects
+				(font
+					(size 1.27 1.27)
+				)
+			)
+		)
+		(property "Value" "Conn_02x03_Counter_Clockwise"
+			(at 106.68 203.2 0)
+			(effects
+				(font
+					(size 1.27 1.27)
+				)
+			)
+		)
+		(property "Footprint" "Connector_PinHeader_2.54mm:PinHeader_2x03_P2.54mm_Vertical"
+			(at 105.41 209.55 0)
+			(effects
+				(font
+					(size 1.27 1.27)
+				)
+				(hide yes)
+			)
+		)
+		(property "Datasheet" "~"
+			(at 105.41 209.55 0)
+			(effects
+				(font
+					(size 1.27 1.27)
+				)
+				(hide yes)
+			)
+		)
+		(property "Description" "Generic connector, double row, 02x03, counter clockwise pin numbering scheme (similar to DIP package numbering), script generated (kicad-library-utils/schlib/autogen/connector/)"
+			(at 105.41 209.55 0)
+			(effects
+				(font
+					(size 1.27 1.27)
+				)
+				(hide yes)
+			)
+		)
+		(pin "3"
+		)
+		(pin "6"
+		)
+		(pin "5"
+		)
+		(pin "4"
+		)
+		(pin "1"
+		)
+		(pin "2"
+		)
+		(instances
+			(project ""
+				(path "/3e3ff72e-d777-45cf-9299-e91389ff12dd/ec3a94af-cbf2-4645-8611-15dc332be977"
+					(reference "J1")
+					(unit 1)
+				)
+			)
+		)
+	)
+	(symbol
 		(lib_id "power:+5V")
 		(at 33.02 160.02 0)
@@
 	)
 	(symbol
+		(lib_id "power:GND")
+		(at 91.44 218.44 0)
+		(unit 1)
+		(exclude_from_sim no)
+		(in_bom yes)
+		(on_board yes)
+		(dnp no)
+		(fields_autoplaced yes)
+		(property "Reference" "#PWR0118"
+			(at 91.44 224.79 0)
+			(effects
+				(font
+					(size 1.27 1.27)
+				)
+				(hide yes)
+			)
+		)
+		(property "Value" "GND"
+			(at 91.44 223.52 0)
+			(effects
+				(font
+					(size 1.27 1.27)
+				)
+			)
+		)
+		(property "Footprint" ""
+			(at 91.44 218.44 0)
+			(effects
+				(font
+					(size 1.27 1.27)
+				)
+				(hide yes)
+			)
+		)
+		(property "Datasheet" ""
+			(at 91.44 218.44 0)
+			(effects
+				(font
+					(size 1.27 1.27)
+				)
+				(hide yes)
+			)
+		)
+		(property "Description" "Power symbol creates a global label with name \"GND\" , ground"
+			(at 91.44 218.44 0)
+			(effects
+				(font
+					(size 1.27 1.27)
+				)
+				(hide yes)
+			)
+		)
+		(pin "1"
+		)
+		(instances
+			(project "TMotor_Rev0_5_1_Mark_2_NAU_OpenExo"
+				(path "/3e3ff72e-d777-45cf-9299-e91389ff12dd/ec3a94af-cbf2-4645-8611-15dc332be977"
+					(reference "#PWR0118")
+					(unit 1)
+				)
+			)
+		)
+	)
+	(symbol
 		(lib_id "TMotor_Rev0_5_1_Mark_2_NAU_OpenExo-eagle-import:R-US_0207/10")
 		(at 203.2 261.62 90)
@@
 					(unit 1)
 				)
-			)
-		)
-	)
-	(symbol
-		(lib_id "Connector:Conn_01x03_Pin")
-		(at 105.41 209.55 180)
-		(unit 1)
-		(exclude_from_sim no)
-		(in_bom yes)
-		(on_board yes)
-		(dnp no)
-		(fields_autoplaced yes)
-		(property "Reference" "J6"
-			(at 106.68 208.2799 0)
-			(effects
-				(font
-					(size 1.27 1.27)
-				)
-				(justify right)
-			)
-		)
-		(property "Value" "Conn_01x03_Pin"
-			(at 106.68 210.8199 0)
-			(effects
-				(font
-					(size 1.27 1.27)
-				)
-				(justify right)
-			)
-		)
-		(property "Footprint" "Connector_PinHeader_2.54mm:PinHeader_1x03_P2.54mm_Vertical"
-			(at 105.41 209.55 0)
-			(effects
-				(font
-					(size 1.27 1.27)
-				)
-				(hide yes)
-			)
-		)
-		(property "Datasheet" "~"
-			(at 105.41 209.55 0)
-			(effects
-				(font
-					(size 1.27 1.27)
-				)
-				(hide yes)
-			)
-		)
-		(property "Description" "Generic connector, single row, 01x03, script generated"
-			(at 105.41 209.55 0)
-			(effects
-				(font
-					(size 1.27 1.27)
-				)
-				(hide yes)
-			)
-		)
-		(pin "2"
-		)
-		(pin "3"
-		)
-		(pin "1"
-		)
-		(instances
-			(project ""
-				(path "/3e3ff72e-d777-45cf-9299-e91389ff12dd/ec3a94af-cbf2-4645-8611-15dc332be977"
-					(reference "J6")
-					(unit 1)
-				)
